File: fightkeyb-pcb.kicad_pcb (KiCad board)
At the start: 2 copper layers, 221.5 x 126.2 mm, 47 parts, among them K10 KEYSW, K11 KEYSW, K12 KEYSW, K13 KEYSW, K14 KEYSW, K15 KEYSW, K16 KEYSW, K17 KEYSW, K18 KEYSW, K19 KEYSW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

Commit message: Finished new v0.1
Parts:
- removed K10, K11, K12, K13, K14, K15, K16, K17, K18, K19, K2, K20, K21, K3, K4, K5, K6, K7, K8, K9: KEYSW, keebs:Mx_Alps_100
- removed M2: ARDUINO_PRO_MICRO, SparkFun-Boards:ARDUINO_PRO_MICRO
- removed REF** (x6): MountingHole_2.2mm_M2_Pad, MountingHole:MountingHole_2.2mm_M2_Pad
- added MX1: MX-1U, MX_Alps_Hybrid:MX-1U-NoLED, F.Cu at (37.1, 31.5)
- added MX10: MX-1U, MX_Alps_Hybrid:MX-1U-NoLED, F.Cu at (208.6, 69.6)
- added MX11: MX-1U, MX_Alps_Hybrid:MX-1U-NoLED, F.Cu at (227.6, 69.6)
- added MX12: MX-1U, MX_Alps_Hybrid:MX-1U-NoLED, F.Cu at (246.7, 69.6)
- added MX13: MX-1U, MX_Alps_Hybrid:MX-1U-NoLED, F.Cu at (56.2, 88.7)
- added MX14: MX-1U, MX_Alps_Hybrid:MX-1U-NoLED, F.Cu at (75.2, 88.6)
- added MX15: MX-1U, MX_Alps_Hybrid:MX-1U-NoLED, F.Cu at (94.3, 88.7)
- added MX16: MX-1U, MX_Alps_Hybrid:MX-1U-NoLED, F.Cu at (194.3, 88.6)
- added MX17: MX-1U, MX_Alps_Hybrid:MX-1U-NoLED, F.Cu at (213.4, 88.6)
- added MX18: MX-1U, MX_Alps_Hybrid:MX-1U-NoLED, F.Cu at (232.4, 88.6)
- added MX19: MX-1U, MX_Alps_Hybrid:MX-1U-NoLED, F.Cu at (251.5, 88.6)
- added MX2: MX-1U, MX_Alps_Hybrid:MX-1U-NoLED, F.Cu at (56.2, 31.5)
- added MX20: MX-1U, MX_Alps_Hybrid:MX-1U-NoLED, F.Cu at (101.4, 126.8)
- added MX3: MX-1U, MX_Alps_Hybrid:MX-1U-NoLED, F.Cu at (75.2, 31.5)
- added MX4: MX-1U, MX_Alps_Hybrid:MX-1U-NoLED, F.Cu at (94.3, 31.5)
- added MX5: MX-1U, MX_Alps_Hybrid:MX-1U-NoLED, F.Cu at (265.7, 31.5)
- added MX6: MX-1U, MX_Alps_Hybrid:MX-1U-NoLED, F.Cu at (51.4, 69.6)
- added MX7: MX-1U, MX_Alps_Hybrid:MX-1U-NoLED, F.Cu at (70.5, 69.6)
- added MX8: MX-1U, MX_Alps_Hybrid:MX-1U-NoLED, F.Cu at (89.5, 69.6)
- added MX9: MX-1U, MX_Alps_Hybrid:MX-1U-NoLED, F.Cu at (189.5, 69.6)
- added SW1: SW_SPST, Keebio-Parts:SW_Tactile_SPST_Angled_MJTP1117, B.Cu at (170.5, 26.8)
- added U1: ProMicro, Keebio-Parts:ArduinoProMicro-BackSide, F.Cu at (151.4, 38.7)
- D1, D10, D11, D12, D13, D14, D15, D16, D17, D18, D19, D2, D20, D3, D4, D5, D6, D7, D8, D9: value D -> D_Small; footprint keyboard_parts:D_SOD123_axial -> Keebio-Parts:Diode-dual
- moved D13 37.2 mm to (58.7, 104.2), turned to 270 degrees
- moved D14 32.4 mm to (77.8, 104.1), turned to 270 degrees
- moved D15 30.0 mm to (96.8, 104.1), turned to 270 degrees
- moved D20 29.2 mm to (118.2, 104.2)
- moved D19 27.9 mm to (256.2, 104.5), turned to 270 degrees
- moved D2 27.1 mm to (58.6, 48.5), turned to 270 degrees
- moved D1 26.9 mm to (39.8, 48.6), turned to 270 degrees
- moved D18 23.6 mm to (235.1, 104.6), turned to 270 degrees
- moved D3 22.4 mm to (77.6, 48.5), turned to 270 degrees
- moved D7 20.2 mm to (72.9, 53.8), turned to 90 degrees
- moved D4 20.1 mm to (96.7, 47.3), turned to 270 degrees
- moved D17 18.8 mm to (215.7, 104.5), turned to 270 degrees
- moved D8 17.7 mm to (91.9, 54.5), turned to 90 degrees
- moved D11 17.7 mm to (230.3, 53.6), turned to 90 degrees
- moved D9 15.7 mm to (198.7, 52.8), turned to 90 degrees
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Routing:
- net Net-(MX15-Pad1): track 0.00 -> 188.4 mm
- net Net-(MX12-Pad1): track 0.00 -> 159.4 mm, vias 0 -> 2
- net Net-(MX13-Pad1): track 0.00 -> 158.6 mm
- net Net-(MX14-Pad1): track 0.00 -> 150.9 mm, vias 0 -> 2
- net Net-(K14-Pad1): track 143.0 -> 0.00 mm
- net Net-(K16-Pad1): track 139.3 -> 0.00 mm, vias 2 -> 0
- net Net-(K15-Pad1): track 120.4 -> 0.00 mm
- net Net-(MX1-Pad1): track 0.00 -> 118.7 mm
- net Net-(K2-Pad1): track 106.8 -> 0.00 mm
- net Net-(MX11-Pad1): track 0.00 -> 95.0 mm, vias 0 -> 1
- net Net-(K12-Pad1): track 88.5 -> 0.00 mm
- net Net-(MX10-Pad1): track 0.00 -> 75.9 mm, vias 0 -> 1
- net Net-(D13-Pad1): track 211.6 -> 274.9 mm, vias 1 -> 0
- net Net-(K13-Pad1): track 57.2 -> 0.00 mm, vias 1 -> 0
- net Net-(MX16-Pad1): track 0.00 -> 54.8 mm
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Other:
- board size 221.5 x 126.2 mm -> 247.6 x 114.3 mm
- rule pad_to_mask_clearance: 0.051 -> 0
- board text added: "hcf hp"
- board text added: "http://coredump.io"
- board text removed: "by coredump"
- board text removed: "gnd"
- board text removed: "rst"

Commit message: Before trying a reroute
Parts:
- added C1: C_Small, Capacitor_SMD:C_0805_2012Metric_Pad1.15x1.40mm_HandSolder, B.Cu at (31.2, 38.0)
- added C10: C_Small, Capacitor_SMD:C_0805_2012Metric_Pad1.15x1.40mm_HandSolder, B.Cu at (202.9, 76.3)
- added C11: C_Small, Capacitor_SMD:C_0805_2012Metric_Pad1.15x1.40mm_HandSolder, B.Cu at (222.2, 76.3)
- added C12: C_Small, Capacitor_SMD:C_0805_2012Metric_Pad1.15x1.40mm_HandSolder, B.Cu at (241.4, 76.3)
- added C13: C_Small, Capacitor_SMD:C_0805_2012Metric_Pad1.15x1.40mm_HandSolder, B.Cu at (50.9, 95.8)
- added C14: C_Small, Capacitor_SMD:C_0805_2012Metric_Pad1.15x1.40mm_HandSolder, B.Cu at (69.7, 95.3)
- added C15: C_Small, Capacitor_SMD:C_0805_2012Metric_Pad1.15x1.40mm_HandSolder, B.Cu at (87.9, 95.3)
- added C16: C_Small, Capacitor_SMD:C_0805_2012Metric_Pad1.15x1.40mm_HandSolder, B.Cu at (188.9, 95.3)
- added C17: C_Small, Capacitor_SMD:C_0805_2012Metric_Pad1.15x1.40mm_HandSolder, B.Cu at (207.7, 95.3)
- added C18: C_Small, Capacitor_SMD:C_0805_2012Metric_Pad1.15x1.40mm_HandSolder, B.Cu at (226.7, 95.5)
- added C19: C_Small, Capacitor_SMD:C_0805_2012Metric_Pad1.15x1.40mm_HandSolder, B.Cu at (245.7, 95.3)
- added C2: C_Small, Capacitor_SMD:C_0805_2012Metric_Pad1.15x1.40mm_HandSolder, B.Cu at (49.4, 37.8)
- added C20: C_Small, Capacitor_SMD:C_0805_2012Metric_Pad1.15x1.40mm_HandSolder, B.Cu at (94.4, 133.3)
- added C3: C_Small, Capacitor_SMD:C_0805_2012Metric_Pad1.15x1.40mm_HandSolder, B.Cu at (69.7, 38.0)
- added C4: C_Small, Capacitor_SMD:C_0805_2012Metric_Pad1.15x1.40mm_HandSolder, B.Cu at (88.9, 38.0)
- added C5: C_Small, Capacitor_SMD:C_0805_2012Metric_Pad1.15x1.40mm_HandSolder, B.Cu at (259.9, 38.0)
- added C6: C_Small, Capacitor_SMD:C_0805_2012Metric_Pad1.15x1.40mm_HandSolder, B.Cu at (45.4, 76.3)
- added C7: C_Small, Capacitor_SMD:C_0805_2012Metric_Pad1.15x1.40mm_HandSolder, B.Cu at (63.9, 76.0)
- added C8: C_Small, Capacitor_SMD:C_0805_2012Metric_Pad1.15x1.40mm_HandSolder, B.Cu at (83.9, 76.0)
- added C9: C_Small, Capacitor_SMD:C_0805_2012Metric_Pad1.15x1.40mm_HandSolder, B.Cu at (183.4, 76.1)
- added D21: WS2812B, Sparkfun Leds:WS2812B, F.Cu at (37.2, 38.0)
- added D22: WS2812B, Sparkfun Leds:WS2812B, F.Cu at (56.2, 38.0)
- added D23: WS2812B, Sparkfun Leds:WS2812B, F.Cu at (75.2, 38.0)
- added D24: WS2812B, Sparkfun Leds:WS2812B, F.Cu at (94.3, 38.0)
- added D25: WS2812B, Sparkfun Leds:WS2812B, F.Cu at (265.7, 38.0)
- added D26: WS2812B, Sparkfun Leds:WS2812B, F.Cu at (51.4, 76.3)
- added D27: WS2812B, Sparkfun Leds:WS2812B, F.Cu at (70.5, 76.3)
- added D28: WS2812B, Sparkfun Leds:WS2812B, F.Cu at (89.5, 76.3)
- added D29: WS2812B, Sparkfun Leds:WS2812B, F.Cu at (189.6, 76.3)
- added D30: WS2812B, Sparkfun Leds:WS2812B, F.Cu at (208.6, 76.3)
- added D31: WS2812B, Sparkfun Leds:WS2812B, F.Cu at (227.7, 76.3)
- added D32: WS2812B, Sparkfun Leds:WS2812B, F.Cu at (246.7, 76.3)
- added D33: WS2812B, Sparkfun Leds:WS2812B, F.Cu at (56.2, 95.8)
- added D34: WS2812B, Sparkfun Leds:WS2812B, F.Cu at (75.2, 95.3)
- added D35: WS2812B, Sparkfun Leds:WS2812B, F.Cu at (94.3, 95.3)
- added D36: WS2812B, Sparkfun Leds:WS2812B, F.Cu at (194.3, 95.3)
- added D37: WS2812B, Sparkfun Leds:WS2812B, F.Cu at (213.4, 95.3)
- added D38: WS2812B, Sparkfun Leds:WS2812B, F.Cu at (232.4, 95.3)
- added D39: WS2812B, Sparkfun Leds:WS2812B, F.Cu at (251.5, 95.3)
- added D40: WS2812B, Sparkfun Leds:WS2812B, F.Cu at (101.4, 133.5)
- added R1: R_Small_US, Keebio-Parts:Resistor-Hybrid-Back, F.Cu at (139.2, 28.3)
Connections:
- U1 pad 20: Net-(U1-Pad20) -> /Led Matrix/DIN
- U1 pad 21: Net-(U1-Pad21) -> /Led Matrix/VCC
- U1 pad 3: Net-(U1-Pad3) -> /Led Matrix/GND
Routing:
- net /Led Matrix/VCC: track 0.00 -> 668.0 mm, vias 0 -> 8
- net Net-(D32-Pad2): track 0.00 -> 267.2 mm
- net Net-(D25-Pad2): track 0.00 -> 260.0 mm, vias 0 -> 4
- net Net-(D39-Pad2): track 0.00 -> 179.7 mm, vias 0 -> 2
- net Net-(D24-Pad2): track 0.00 -> 169.6 mm, vias 0 -> 2
- net Net-(D21-Pad4): track 0.00 -> 116.9 mm, vias 0 -> 1
- net Net-(D28-Pad2): track 0.00 -> 115.5 mm
- net Net-(D35-Pad2): track 0.00 -> 100.5 mm, vias 0 -> 2
- net Net-(MX13-Pad1): track 158.6 -> 217.6 mm
- net Net-(D1-Pad2): track 17.8 -> 48.5 mm
- net /Led Matrix/GND: track 0.00 -> 23.1 mm, vias 0 -> 2
- net Net-(MX10-Pad1): track 75.9 -> 97.0 mm
- net /Led Matrix/DIN: track 0.00 -> 21.0 mm
- net Net-(D3-Pad2): track 17.6 -> 38.5 mm
- net Net-(D19-Pad2): track 17.4 -> 0.00 mm
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- added copper zone on B.Cu, net /Led Matrix/GND
- added copper zone on F.Cu, net /Led Matrix/GND

Commit message: Finished first production test
Parts:
- added ?: MountingHole_4.3mm_M4, MountingHole:MountingHole_4.3mm_M4, F.Cu at (152.5, 71.4)
- C1, C10, C11, C12, C13, C14, C15, C16, C17, C18, C19, C2, C20, C3, C4, C5, C6, C7, C8, C9: value C_Small -> 0u1
- D1, D10, D11, D12, D13, D14, D15, D16, D17, D18, D19, D2, D20, D3, D4, D5, D6, D7, D8, D9: value D_Small -> 1N4148; footprint Keebio-Parts:Diode-dual -> Diode_SMD:D_0805_2012Metric_Pad1.15x1.40mm_HandSolder
- R1: value R_Small_US -> 330R; footprint Keebio-Parts:Resistor-Hybrid-Back -> Resistor_SMD:R_0805_2012Metric_Pad1.15x1.40mm_HandSolder
- moved R1 49.1 mm to (184.9, 46.0)
- moved D20 26.1 mm to (109.4, 128.8)
- moved D12 24.8 mm to (254.7, 72.3)
- moved D9 19.5 mm to (197.4, 72.3)
- moved D10 19.5 mm to (216.7, 72.3)
- moved D11 19.4 mm to (235.7, 72.3)
- moved D6 19.0 mm to (59.4, 71.8)
- moved SW1 19.0 mm to (189.5, 26.8)
- moved U1 19.0 mm to (170.4, 38.7)
- moved D7 18.8 mm to (78.4, 71.8)
- moved D8 18.2 mm to (97.4, 71.8)
- moved D1 16.0 mm to (45.2, 33.5), turned to 90 degrees
- moved D2 16.0 mm to (64.2, 33.6), turned to 90 degrees
- moved D3 16.0 mm to (83.2, 33.5), turned to 90 degrees
- moved D4 14.9 mm to (102.2, 33.5), turned to 90 degrees
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Connections:
- D26 pad 4: Net-(D25-Pad2) -> Net-(D21-Pad4)
- D33 pad 4: Net-(D32-Pad2) -> Net-(D21-Pad4)
- D40 pad 4: Net-(D39-Pad2) -> Net-(D21-Pad4)
- SW1 pad 1: Net-(SW1-Pad1) -> /Led Matrix/GND
- U1 pad 23: Net-(SW1-Pad1) -> /Led Matrix/GND
- U1 pad 4: Net-(U1-Pad4) -> /Led Matrix/GND
Routing:
- net Net-(D32-Pad2): track 267.2 -> 0.00 mm
- net Net-(D39-Pad2): track 179.7 -> 1.18 mm, vias 2 -> 0
- net Net-(D21-Pad4): track 116.9 -> 283.1 mm, vias 1 -> 2
- net /Led Matrix/VCC: track 668.0 -> 723.4 mm, vias 8 -> 20
- net Net-(D10-Pad1): track 176.6 -> 225.0 mm
- net Net-(D1-Pad2): track 48.5 -> 7.78 mm
- net Net-(D20-Pad1): track 65.2 -> 105.6 mm
- net Net-(MX10-Pad1): track 97.0 -> 63.1 mm, vias 1 -> 0
- net Net-(MX13-Pad1): track 217.6 -> 184.6 mm
- net Net-(D25-Pad2): track 260.0 -> 228.8 mm, vias 4 -> 6
- net Net-(D3-Pad2): track 38.5 -> 7.72 mm
- net Net-(D2-Pad2): track 34.2 -> 7.76 mm
- net Net-(D13-Pad1): track 274.7 -> 253.4 mm
- net Net-(D28-Pad2): track 115.5 -> 96.2 mm
- net Net-(MX1-Pad1): track 118.7 -> 137.7 mm
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Other:
- board text added: "/u/coredump777"
- board text removed: "http://coredump.io"
